Commit message: Adding resources to READMes, and adding final configs

File: simulation_challenge/urdf/orion_mod.urdf.xacro (robot description, xacro)
@@ -21,4 +21,46 @@
     </xacro:if>
     <xacro:if value="${dummy_sensor}">
+        <link name="dummy_link">
+            <visual>
+                <geometry>
+                    <box size="0.025 0.025 0.025"/>
+                </geometry>
+                <material name="green">
+                    <color rgba="0 1 0 1"/>
+                </material>
+            </visual>
+            <collision>
+                <geometry>
+                    <box size="0.025 0.025 0.025"/>
+                </geometry>
+            </collision>
+            <inertial>
+                <mass value="0.1"/>
+                <inertia ixx="1e-5" ixy="0.0" ixz="0.0"
+                        iyy="1e-5" iyz="0.0"
+                        izz="1e-5"/>
+            </inertial>
+        </link>
+        <!-- Fixed joint connecting to base_link -->
+        <joint name="dummy_link_joint" type="fixed">
+            <parent link="base_link"/>
+            <child link="dummy_link"/>
+            <origin xyz="-0.05 0 0.32" rpy="0 0 0"/> <!-- You can change the pose -->
+        </joint>
+        <gazebo>
+            <!-- System plugin to handle Dummy Sensors-->
+            <plugin
+                filename="DummySensorSystem"
+                name="custom::DummySensorSystem">
+            </plugin>
+        </gazebo>
+        <gazebo reference="dummy_link">
+            <!-- Dummy Sensor Definition -->
+            <sensor name="my_dummy" type="custom" gz:type="dummy" xmlns:gz="http://gazebosim.org/schema">
+                <always_on>1</always_on>
+                <update_rate>30</update_rate>
+                <visualize>true</visualize>
+            </sensor>
+        </gazebo>
     </xacro:if>
 </robot>

Commit message: Fixing Dummy Sensor as the problem was that it required a ISystemConfigure implementation

File: simulation_challenge/urdf/orion_mod.urdf.xacro (robot description, xacro)
@@ -6,4 +6,6 @@
     <xacro:property name="rasp" default="rpi4"/>
     <xacro:property name="gazebo" default="true"/>
+    <xacro:property name="simplified" default="true"/>
+    <xacro:property name="motor" default="100"/>
     <xacro:property name="ros2_control" default="false"/>
     <xacro:property name="dummy_sensor" default="$(arg dummy_sensor)"/>
@@ -61,4 +63,5 @@
                 <update_rate>30</update_rate>
                 <visualize>true</visualize>
+                <gz:dummy>GSOC_2025</gz:dummy>
             </sensor>
         </gazebo>
